Commit message: 将小腿collision模型下半部截掉

File: source/direct_pm01_walk/direct_pm01_walk/assets/robots/pm01/urdf/pm01.urdf (robot description, URDF)
Before this commit: robot pm01, 25 links, 24 joints
Links:
- link link_ankle_pitch_l: geometry visual mesh filename=../meshes/link_ankle_pitch_l.stl
- link link_ankle_pitch_r: geometry visual mesh filename=../meshes/link_ankle_pitch_r.stl
- link link_knee_pitch_l: geometry collision mesh filename=../meshes/link_knee_pitch_l_collision.stl; visual mesh filename=../meshes/link_knee_pitch_l.stl
- link link_knee_pitch_r: geometry collision mesh filename=../meshes/link_knee_pitch_r_collision.stl; visual mesh filename=../meshes/link_knee_pitch_r.stl
